Commit message: update 6 files and delete 1 file

File: urdf/SLIP_Model.urdf (robot description, URDF)
Before this commit: robot Assem4, 3 links, 2 joints
Links:
- removed link Spring_Link
- link mass_Link: mass 1 -> 1.5
Joints:
- removed joint Spring_joint
- joint mass_joint: axis 0 0 0 -> 0 0 -1; limit (none) -> lower=0 upper=0 effort=0 velocity=0; origin xyz=0 0 1 rpy=0 0 0 -> xyz=0 0 1.1 rpy=0 0 0; type fixed -> prismatic

Commit message: update Pybullet_Simulation.py and SLIP_Model.urdf

File: urdf/SLIP_Model.urdf (robot description, URDF)
Before this commit: robot Assem1, 2 links, 1 joints
Joints:
- joint mass_joint: limit lower=0 upper=0 effort=0 velocity=0 -> lower=0 upper=1 effort=0 velocity=0
